Commit message: fixed lidar issues

File: urdf/elea_diff_robot.urdf (robot description, URDF)
Before this commit: robot elea_diff_robot, 5 links, 4 joints
Links:
- added link apf_front_center; visual sphere radius=0.02
- added link apf_front_left; visual sphere radius=0.02
- added link apf_front_right; visual sphere radius=0.02
- added link apf_left_side; visual sphere radius=0.02
- added link apf_rear_center; visual sphere radius=0.02
- added link apf_right_side; visual sphere radius=0.02
- added link lidar_link, mass 0.1; collision cylinder length=0.05 radius=0.03; visual cylinder length=0.05 radius=0.03
- link base_link: geometry collision box size=1.849 1.445 0.51025; visual box size=1.849 1.445 0.51025
Joints:
- added joint apf_front_center_joint: type fixed, parent base_link, child apf_front_center, origin xyz=0.9245 0 0 rpy=0 0 0
- added joint apf_front_left_joint: type fixed, parent base_link, child apf_front_left, origin xyz=0.8 0.6 0 rpy=0 0 0
- added joint apf_front_right_joint: type fixed, parent base_link, child apf_front_right, origin xyz=0.8 -0.6 0 rpy=0 0 0
- added joint apf_left_side_joint: type fixed, parent base_link, child apf_left_side, origin xyz=0 0.7225 0 rpy=0 0 0
- added joint apf_rear_center_joint: type fixed, parent base_link, child apf_rear_center, origin xyz=-0.9245 0 0 rpy=0 0 0
- added joint apf_right_side_joint: type fixed, parent base_link, child apf_right_side, origin xyz=0 -0.7225 0 rpy=0 0 0
- added joint lidar_joint: type fixed, parent base_link, child lidar_link, origin xyz=0 0 0.255125 rpy=0 0 0
- joint front_support_joint: origin xyz=0.9245 0 -0.54025 rpy=0 0 0 -> xyz=0.9245 0 -0.285125 rpy=0 0 0
- joint left_wheel_joint: origin xyz=0 0.7425 -0.51025 rpy=1.5708 0 0 -> xyz=0 0.7425 -0.255125 rpy=1.5708 0 0
- joint rear_support_joint: origin xyz=-0.9245 0 -0.54025 rpy=0 0 0 -> xyz=-0.9245 0 -0.285125 rpy=0 0 0
- joint right_wheel_joint: origin xyz=0 -0.7425 -0.51025 rpy=1.5708 0 0 -> xyz=0 -0.7425 -0.255125 rpy=1.5708 0 0

Commit message: robot detectando y moviendose

File: urdf/elea_diff_robot.urdf (robot description, URDF)
Before this commit: robot elea_diff_robot, 12 links, 11 joints
Links:
- removed link apf_front_left
- removed link apf_front_right
- removed link apf_left_side
- removed link apf_rear_center
- removed link apf_right_side
Joints:
- removed joint apf_front_left_joint
- removed joint apf_front_right_joint
- removed joint apf_left_side_joint
- removed joint apf_rear_center_joint
- removed joint apf_right_side_joint

Commit message: minor changes

File: urdf/elea_diff_robot.urdf (robot description, URDF)
Before this commit: robot elea_diff_robot, 7 links, 6 joints
Links:
- link apf_front_center: geometry 
Joints:
- removed joint apf_front_center_joint
- added joint apf_left_center_joint: type fixed, parent base_link, child apf_left_center, origin xyz=0 0.7225 0.255125 rpy=0 0 1.5708

Commit message: added kmp mesh and adjusted dimensions

File: urdf/elea_diff_robot.urdf (robot description, URDF)
Before this commit: robot elea_diff_robot, 7 links, 6 joints
Links:
- added link apf_left_center
- link base_link: geometry collision box size=1.08 0.63 0.7; visual mesh filename=package://elea_amr/urdf/KMP200.dae scale=1 1 1
Joints:
- added joint apf_front_center_joint: type fixed, parent base_link, child apf_front_center, origin xyz=0.54 0 0.35 rpy=0 0 0
- joint apf_left_center_joint: origin xyz=0 0.7225 0.255125 rpy=0 0 1.5708 -> xyz=0 0.315 0.35 rpy=0 0 1.5708
- joint front_support_joint: origin xyz=0.9245 0 -0.285125 rpy=0 0 0 -> xyz=0.54 0 -0.38 rpy=0 0 0
- joint left_wheel_joint: origin xyz=0 0.7425 -0.255125 rpy=1.5708 0 0 -> xyz=0 0.315 -0.35 rpy=1.5708 0 0
- joint lidar_joint: origin xyz=0 0 0.255125 rpy=0 0 0 -> xyz=0 0 0.35 rpy=0 0 0
- joint rear_support_joint: origin xyz=-0.9245 0 -0.285125 rpy=0 0 0 -> xyz=-0.54 0 -0.38 rpy=0 0 0
- joint right_wheel_joint: origin xyz=0 -0.7425 -0.255125 rpy=1.5708 0 0 -> xyz=0 -0.315 -0.35 rpy=1.5708 0 0

Commit message: simulation in dev container with digilab

File: urdf/elea_diff_robot.urdf (robot description, URDF)
Before this commit: robot elea_diff_robot, 8 links, 7 joints
Links:
- link base_link: geometry collision box size=1.08 0.63 0.7; visual mesh filename=file:///workspaces/elea_ws/install/elea_amr/share/elea_amr/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 scale=1 1 1

Commit message: change of wheels to correct the movement of the robot (al revez)

File: urdf/elea_diff_robot.urdf (robot description, URDF)
Before this commit: robot elea_diff_robot, 8 links, 7 joints
Links:
- removed link apf_front_center
- removed link apf_left_center
- added link apf_front_left_corner
- added link apf_front_right_corner
- added link apf_rear_left_corner
- added link apf_rear_right_corner
- added link base_link_rotado
Joints:
- removed joint apf_front_center_joint
- removed joint apf_left_center_joint
- added joint apf_front_left_corner_joint: type fixed, parent base_link, child apf_front_left_corner, origin xyz=0.54 0.315 0.35 rpy=0 0 0
- added joint apf_front_right_corner_joint: type fixed, parent base_link, child apf_front_right_corner, origin xyz=0.54 -0.315 0.35 rpy=0 0 0
- added joint apf_rear_left_corner_joint: type fixed, parent base_link, child apf_rear_left_corner, origin xyz=-0.54 0.315 0.35 rpy=0 0 0
- added joint apf_rear_right_corner_joint: type fixed, parent base_link, child apf_rear_right_corner, origin xyz=-0.54 -0.315 0.35 rpy=0 0 0
- added joint joint_base_link_rotada: type fixed, parent base_link, child base_link_rotado, origin xyz=0 0 0 rpy=0 0 3.1416
- joint left_wheel_joint: parent base_link -> base_link_rotado
- joint right_wheel_joint: parent base_link -> base_link_rotado
